File: pcb/ESPhome_greenhouse_controller/ESPhome_greenhouse_controller.kicad_pcb (KiCad board)
At the start: 2 copper layers, 8 parts, among them K1 SANYOU_SRD_Form_C, K2 SANYOU_SRD_Form_C, K3 SANYOU_SRD_Form_C, K4 SANYOU_SRD_Form_C, K5 SANYOU_SRD_Form_C, K6 SANYOU_SRD_Form_C, U1 PC817, U2 PC817

Commit message: update
Parts:
- added D1: SM4007, Diode_SMD:D_MELF, F.Cu at (70.2, 42.2)
- added D2: SM4007, Diode_SMD:D_MELF, F.Cu at (70.2, 46.5)
- added F2: Polyfuse, Fuse:Fuse_Bourns_MF-RHT1100, F.Cu at (133.8, 56.8)
- added R1: 50mR, Resistor_SMD:R_1206_3216Metric, F.Cu at (155.5, 70.7)
- added R2: 50mR, Resistor_SMD:R_1206_3216Metric, F.Cu at (155.5, 74.0)
- added U3: INA219AxD, Package_SO:SOIC-8_3.9x4.9mm_P1.27mm, F.Cu at (147.8, 77.3)
- added U4: INA219AxD, Package_SO:SOIC-8_3.9x4.9mm_P1.27mm, F.Cu at (147.8, 83.9)
Connections:
- K1 pad 2: +12V -> +24V
- K1 pad 3: VBUS -> Net-(U3-IN+)
- K2 pad 2: +12V -> +24V
- K2 pad 3: VBUS -> Net-(U3-IN+)
- K3 pad 2: +12V -> +24V
- K3 pad 3: VBUS -> Net-(U4-IN+)
- K4 pad 2: +12V -> +24V
- K4 pad 3: VBUS -> Net-(U4-IN+)
- K5 pad 2: +12V -> +24V
- K5 pad 3: VBUS -> +24V
- K6 pad 2: +12V -> +24V
- K6 pad 3: VBUS -> +24V
