File: pcb/_autosave-ESPhome_greenhouse_controller.kicad_sch (KiCad schematic)
At the start: 53 parts, among them K1 SANYOU_SRD_Form_C, K2 SANYOU_SRD_Form_C, K3 SANYOU_SRD_Form_C, K4 SANYOU_SRD_Form_C, K5 SANYOU_SRD_Form_C, K6 SANYOU_SRD_Form_C, U1 EL817, U10 LTV-817S, U11 LTV-817S, U12 LTV-817S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

Commit message: update
Parts:
- added U14: STM32F103CBTx, Package_QFP:LQFP-48_7x7mm_P0.5mm, symbol MCU_ST_STM32F1:STM32F103CBTx
Connections:
- net +24V: now also U3.8 (IN+), U4.8 (IN+); no longer K2.1, MOD1.A12, U3.7 (IN-), U4.7 (IN-)
- net at K1.3, K2.3, R1.2: now also U3.7 (IN-); no longer U3.8 (IN+)
- net at K3.3, K4.3, R2.2: now also U4.7 (IN-); no longer U4.8 (IN+)
- new net: U14.23 (VSS), U14.35 (VSS), U14.47 (VSS)
- new net M1-: K2.1, MOD1.A12
Other:
- moved on the sheet: U3, U4
