File: pcb/ESPhome_greenhouse_controller.kicad_sch (KiCad schematic)
At the start: 53 parts, among them K1 SANYOU_SRD_Form_C, K2 SANYOU_SRD_Form_C, K3 SANYOU_SRD_Form_C, K4 SANYOU_SRD_Form_C, K5 SANYOU_SRD_Form_C, K6 SANYOU_SRD_Form_C, U1 EL817, U10 LTV-817S, U11 LTV-817S, U12 LTV-817S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

Commit message: update
Parts:
- removed U1, U2: EL817, Package_DIP:DIP-4_W7.62mm, symbol Isolator:EL817
- added U1, U15: LTV-817S, Package_DIP:SMDIP-4_W9.53mm, symbol Isolator:LTV-817S
- added U14: STM32F103CBTx, Package_QFP:LQFP-48_7x7mm_P0.5mm, symbol MCU_ST_STM32F1:STM32F103CBTx
Connections:
- net +24V: now also MOD1.B10, MOD1.B12, MOD1.B6, MOD1.B8, U3.8 (IN+), U4.8 (IN+); no longer K2.1, MOD1.A12, U3.7 (IN-), U4.7 (IN-)
- net +3V3: now also U1.1, U14.1 (VBAT), U14.24 (VDD), U14.36 (VDD), U14.48 (VDD), U14.9 (VDDA), U15.1
- net GND: now also U14.23 (VSS), U14.35 (VSS), U14.47 (VSS), U14.8 (VSSA)
- net GND2: now also U1.3, U15.3
- net IN3_1_P: now also MOD1.B11
- net IN3_2_P: now also MOD1.B9
- net IN4_1_P: now also MOD1.B7
- net IN4_2_P: now also MOD1.B5
- net SIG_CLOSE: now also U15.4
- net SIG_OPEN: now also U1.4
- net nSIG_CLOSE: now also U15.2
- net nSIG_OPEN: now also U1.2
- net at K1.3, K2.3, R1.2: now also U3.7 (IN-); no longer U3.8 (IN+)
- net at K3.3, K4.3, R2.2: now also U4.7 (IN-); no longer U4.8 (IN+)
- new net M1-: K2.1, MOD1.A12
Other:
- moved on the sheet: U3, U4

Commit message: update
Parts:
- added J1, J2: Conn_01x04_Pin, symbol 380-015-113L001:Conn_01x04_Pin
- added R27: R0603_10k_1%_100mW_100PPM_AC, Resistor_SMD:R_0603_1608Metric, symbol Resistors_SMD_0603:R0603_10k_1%_100mW_100PPM_AC
Connections:
- net P-UP is gone; now on net +3V3: R10.1, R15.1, R16.1, R21.1, R22.1, R3.1, R4.1, R9.1
- net +3V3: now also J1.1 (Pin_1), J2.1 (Pin_1)
- net GND: now also J1.4 (Pin_4), J2.4 (Pin_4), R27.2
- net IN3_1_L: now also U14.18 (PB0)
- net IN3_2_L: now also U14.19 (PB1)
- net SCL: now also U14.42 (PB6)
- net SDA: now also U14.43 (PB7)
- net IN4_1_L: now reaches U14.20 (PB2)
- net IN4_1_L: now also R21.2, U12.4
- net TX: now reaches U14.30 (PA9)
- net TX: now also J1.3 (Pin_3), J2.3 (Pin_3)
- net RX: now reaches U14.31 (PA10)
- net RX: now also J1.2 (Pin_2), J2.2 (Pin_2)
- net SWDIO: now reaches U14.34 (PA13)
- net SWCLK: now reaches U14.37 (PA14)
- net IN4_2_L: now reaches U14.39 (PB3)
- net IN4_2_L: now also R22.2, U13.4
- net IN2_1_L: now reaches U14.40 (PB4)
- net IN2_1_L: now also R9.2, U8.4
- net IN2_2_L: now reaches U14.41 (PB5)
- net IN2_2_L: now also R10.2, U9.4
- net BOOT0: now reaches U14.44 (BOOT0)
- net BOOT0: now also R27.1
- net IN1_1_L: now reaches U14.45 (PB8)
- net IN1_1_L: now also R3.2, U6.4
- net IN1_2_L: now reaches U14.46 (PB9)
- net IN1_2_L: now also R4.2, U7.4
- net NRST: now reaches U14.7 (NRST)
- removed net IN1_L: R21.2, R3.2, R9.2, U12.4, U6.4, U8.4
- removed net IN2_L: R10.2, R22.2, R4.2, U13.4, U7.4, U9.4
Other:
- moved on the sheet: U14

Commit message: update
Parts:
- removed U14: STM32F103CBTx, Package_QFP:LQFP-48_7x7mm_P0.5mm, symbol MCU_ST_STM32F1:STM32F103CBTx
- removed U3, U4: INA219AxD, Package_SO:SOIC-8_3.9x4.9mm_P1.27mm, symbol Sensor_Energy:INA219AxD
- added U14, U3: INA237, Package_SO:VSSOP-10_3x3mm_P0.5mm, symbol Sensor_Energy:INA237
- added U2: MCP23017_SO, Package_SO:SOIC-28W_7.5x17.9mm_P1.27mm, symbol Interface_Expansion:MCP23017_SO
Connections:
- net +24V: now also U14.10 (Vin+), U14.8 (Vbus), U3.10 (Vin+), U3.8 (Vbus)
- net +3V3: now also U14.6 (VS), U2.9 (VDD), U3.2 (A0), U3.6 (VS)
- net GND: now also U14.1 (A1), U14.2 (A0), U14.7 (GND), U2.10 (VSS), U3.1 (A1), U3.7 (GND)
- net IN1_1_L: now also U2.21 (GPA0)
- net IN1_2_L: now also U2.22 (GPA1)
- net IN2_1_L: now also U2.5 (GPB4)
- net IN2_2_L: now also U2.6 (GPB5)
- net IN3_1_L: now also U2.1 (GPB0)
- net IN3_2_L: now also U2.2 (GPB1)
- net IN4_1_L: now also U2.3 (GPB2)
- net IN4_2_L: now also U2.4 (GPB3)
- net SCL: now also U14.5 (SCL), U2.12 (SCK), U3.5 (SCL)
- net SDA: now also U14.4 (SDA), U2.13 (SDA), U3.4 (SDA)
- net nFWD1: now also D1.2 (A), K1.5, U5.11 (O6); no longer D2.2 (A), K2.5, U5.12 (O5)
- net nREV1: now also D2.2 (A), K2.5, U5.12 (O5); no longer D1.2 (A), K1.5, U5.11 (O6)
- net at K1.3, K2.3, R1.2: now also U14.9 (Vin-)
- net at K3.3, K4.3, R2.2: now also U3.9 (Vin-)
- new net M1_A: U14.3 (~{Alert})
- new net M2_A: U3.3 (~{Alert})
Other:
- moved on the sheet: MOD1C, MOD1D

Commit message: update
Parts:
- added U4: MCP23017_SO, Package_SO:SOIC-28W_7.5x17.9mm_P1.27mm, symbol Interface_Expansion:MCP23017_SO
Connections:
- net +3V3: now also U4.9 (VDD)
- net GND: now also U4.10 (VSS)
- net M1_A: now also U2.7 (GPB6)
- net M2_A: now also U2.23 (GPA2)
- net SCL: now also U4.12 (SCK)
- net SDA: now also U4.13 (SDA)
- net LIGHT: now reaches U5.2 (I2)
- net LIGHT: now also U4.1 (GPB0)
- net FWD2: now reaches U5.3 (I3)
- net FWD2: now also U4.2 (GPB1)
- net REV2: now reaches U5.4 (I4)
- net REV2: now also U4.3 (GPB2)
- net REV1: now reaches U5.5 (I5)
- net REV1: now also U4.4 (GPB3)
- net FWD1: now reaches U5.6 (I6)
- net FWD1: now also U4.5 (GPB4)
- net SOUND: now reaches U5.7 (I7)
- net SOUND: now also U4.6 (GPB5)
Other:
- moved on the sheet: MOD1C, MOD1D
