File: pcb/ESPhome_greenhouse_controller.kicad_sch (KiCad schematic)
At the start: 58 parts, among them J1 Conn_01x04_Pin, J2 Conn_01x04_Pin, K1 SANYOU_SRD_Form_C, K2 SANYOU_SRD_Form_C, K3 SANYOU_SRD_Form_C, K4 SANYOU_SRD_Form_C, K5 SANYOU_SRD_Form_C, K6 SANYOU_SRD_Form_C, U1 LTV-817S, U10 LTV-817S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

Commit message: update
Parts:
- removed R27: R0603_10k_1%_100mW_100PPM_AC, Resistor_SMD:R_0603_1608Metric, symbol Resistors_SMD_0603:R0603_10k_1%_100mW_100PPM_AC
Connections:
- net INT: now reaches U4.19 (INTB)
- net INT: now also U2.19 (INTB), U2.20 (INTA), U4.20 (INTA)
Changed lines of the file:
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@@
 	)
 	(junction
+		(at 158.75 173.99)
+		(diameter 0)
+		(color 0 0 0 0)
+	)
+	(junction
 		(at 347.98 106.68)
 		(diameter 0)
@@
 	)
 	(junction
+		(at 158.75 93.98)
+		(diameter 0)
+		(color 0 0 0 0)
+	)
+	(junction
 		(at 67.31 162.56)
 		(diameter 0)
@@
 	(wire
 		(pts
+			(xy 158.75 173.99) (xy 147.32 173.99)
+		)
+		(stroke
+			(width 0)
+			(type default)
+		)
+	)
+	(wire
+		(pts
 			(xy 158.75 78.74) (xy 147.32 78.74)
 		)
@@
 	(wire
 		(pts
-			(xy 111.76 251.46) (xy 111.76 262.89)
-		)
-		(stroke
-			(width 0)
-			(type default)
-		)
-	)
-	(wire
-		(pts
 			(xy 347.98 85.09) (xy 347.98 106.68)
 		)
@@
 	(wire
 		(pts
-			(xy 111.76 270.51) (xy 111.76 276.86)
-		)
-		(stroke
-			(width 0)
-			(type default)
-		)
-	)
-	(wire
-		(pts
 			(xy 289.56 129.54) (xy 289.56 133.35)
 		)
@@
 	(wire
 		(pts
-			(xy 111.76 251.46) (xy 99.06 251.46)
-		)
-		(stroke
-			(width 0)
-			(type default)
-		)
-	)
-	(wire
-		(pts
 			(xy 275.59 129.54) (xy 275.59 134.62)
 		)
@@
 	(wire
 		(pts
+			(xy 158.75 93.98) (xy 147.32 93.98)
+		)
+		(stroke
+			(width 0)
+			(type default)
+		)
+	)
+	(wire
+		(pts
 			(xy 283.21 50.8) (xy 283.21 59.69)
 		)
@@
 	(wire
 		(pts
+			(xy 158.75 91.44) (xy 158.75 93.98)
+		)
+		(stroke
+			(width 0)
+			(type default)
+		)
+	)
+	(wire
+		(pts
 			(xy 347.98 223.52) (xy 341.63 223.52)
 		)
@@
 	(wire
 		(pts
+			(xy 158.75 171.45) (xy 158.75 173.99)
+		)
+		(stroke
+			(width 0)
+			(type default)
+		)
+	)
+	(wire
+		(pts
 			(xy 267.97 271.78) (xy 276.86 271.78)
 		)
@@
 	)
 	(image
-		(at 492.76 36.83)
+		(at -73.66 47.625)
 		(scale 0.324809)
 		(data "iVBORw0KGgoAAAANSUhEUgAABkAAAARDCAYAAAAwB+0gAAAABGdBTUEAALGPC/xhBQAAACBjSFJN"
@@
 		)
 	)
+	(label "INT"
+		(at 147.32 93.98 0)
+		(fields_autoplaced yes)
+		(effects
+			(font
+				(size 1.27 1.27)
+			)
+			(justify left bottom)
+		)
+	)
 	(label "IN4_2_P"
 		(at 21.59 157.48 0)
@@
 		)
 	)
-	(label "BOOT0"
-		(at 99.06 251.46 0)
-		(fields_autoplaced yes)
-		(effects
-			(font
-				(size 1.27 1.27)
-			)
-			(justify left bottom)
-		)
-	)
 	(label "LIGHT"
 		(at 207.01 156.21 180)
@@
 		)
 	)
+	(label "INT"
+		(at 147.32 173.99 0)
+		(fields_autoplaced yes)
+		(effects
+			(font
+				(size 1.27 1.27)
+			)
+			(justify left bottom)
+		)
+	)
 	(label "IN3_2_L"
 		(at 91.44 104.14 180)
@@
 	)
 	(symbol
-		(lib_id "power:GND")
-		(at 111.76 276.86 0)
-		(unit 1)
-		(exclude_from_sim no)
-		(in_bom yes)
-		(on_board yes)
-		(dnp no)
-		(fields_autoplaced yes)
-		(property "Reference" "#PWR040"
-			(at 111.76 283.21 0)
-			(effects
-				(font
-					(size 1.27 1.27)
-				)
-				(hide yes)
-			)
-		)
-		(property "Value" "GND"
-			(at 111.76 281.94 0)
-			(effects
-				(font
-					(size 1.27 1.27)
-				)
-			)
-		)
-		(property "Footprint" ""
-			(at 111.76 276.86 0)
-			(effects
-				(font
-					(size 1.27 1.27)
-				)
-				(hide yes)
-			)
-		)
-		(property "Datasheet" ""
-			(at 111.76 276.86 0)
-			(effects
-				(font
-					(size 1.27 1.27)
-				)
-				(hide yes)
-			)
-		)
-		(property "Description" ""
-			(at 111.76 276.86 0)
-			(effects
-				(font
-					(size 1.27 1.27)
-				)
-				(hide yes)
-			)
-		)
-		(pin "1"
-		)
-		(instances
-			(project "ESPhome_greenhouse_controller"
-				(path "/369bf40f-e28a-46b1-be37-62b35f4960a2"
-					(reference "#PWR040")
-					(unit 1)
-				)
-			)
-		)
-	)
-	(symbol
 		(lib_id "power:+3V3")
 		(at 67.31 181.61 0)
@@
 					(unit 1)
 				)
-			)
-		)
-	)
-	(symbol
-		(lib_id "Resistors_SMD_0603:R0603_10k_1%_100mW_100PPM_AC")
-		(at 111.76 266.7 0)
-		(unit 1)
-		(exclude_from_sim no)
-		(in_bom yes)
-		(on_board yes)
-		(dnp no)
-		(property "Reference" "R27"
-			(at 109.22 267.97 90)
-			(effects
-				(font
-					(size 1.27 1.27)
-				)
-				(justify left)
-			)
-		)
-		(property "Value" "R0603_10k_1%_100mW_100PPM_AC"
-			(at 114.3 261.62 0)
-			(effects
-				(font
-					(size 1.27 1.27)
-				)
-				(justify left)
-				(hide yes)
-			)
-		)
-		(property "Footprint" "Resistor_SMD:R_0603_1608Metric"
-			(at 122.8852 252.73 0)
-			(effects
-				(font
-					(size 1.27 1.27)
-				)
-				(hide yes)
-			)
-		)
-		(property "Datasheet" "http://www.yageo.com/NewPortal/yageodocoutput?fileName=/pdf/R-Chip/PYu-AC_51_RoHS_L_6.pdf"
-			(at 111.76 266.7 0)
-			(effects
-				(font
-					(size 1.27 1.27)
-				)
-				(hide yes)
-			)
-		)
-		(property "Description" "RES SMD 10K OHM 1% 1/10W 0603"
-			(at 121.92 248.92 0)
-			(effects
-				(font
-					(size 1.27 1.27)
-				)
-				(hide yes)
-			)
-		)
-		(property "Value1" "10k"
-			(at 111.76 269.24 90)
-			(effects
-				(font
-					(size 1.27 1.27)
-				)
-				(justify left)
-			)
-		)
-		(property "Manufacturer" "Yageo"
-			(at 121.92 248.92 0)
-			(effects
-				(font
-					(size 1.27 1.27)
-				)
-				(hide yes)
-			)
-		)
-		(property "Manufacturer Part Number" "AC0603FR-0710KL"
-			(at 121.92 248.92 0)
-			(effects
-				(font
-					(size 1.27 1.27)
-				)
-				(hide yes)
-			)
-		)
-		(property "Supplier" "Digi-Key"
-			(at 124.46 256.54 0)
-			(effects
-				(font
-					(size 1.27 1.27)
-				)
-				(hide yes)
-			)
-		)
-		(property "Supplier Part Number" "311-10KLDCT-ND"
-			(at 121.92 248.92 0)
-			(effects
-				(font
-					(size 1.27 1.27)
-				)
-				(hide yes)
-			)
-		)
-		(property "Unit Price" "0.08"
-			(at 121.92 248.92 0)
-			(effects
-				(font
-					(size 1.27 1.27)
-				)
-				(hide yes)
-			)
-		)
-		(property "Package / Case" "R0603"
-			(at 121.92 248.92 0)
-			(effects
-				(font
-					(size 1.27 1.27)
-				)
-				(hide yes)
-			)
-		)
-		(pin "1"
-		)
-		(pin "2"
-		)
-		(instances
-			(project "ESPhome_greenhouse_controller"
-				(path "/369bf40f-e28a-46b1-be37-62b35f4960a2"
-					(reference "R27")
-					(unit 1)
-				)

Commit message: update
Parts:
- added C1, C2: EKM227M1HG1BRRSHP, Capacitor_THT:CP_Radial_D10.0mm_P5.00mm, symbol Device:C_Polarized
- added D7: GBU6D, Diode_THT:Diode_Bridge_Vishay_GBU, symbol Diode_Bridge:GBU6D
Connections:
- net FWD1: now also U4.8 (GPB7); no longer U4.5 (GPB4)
- net FWD2: now also U4.5 (GPB4); no longer U4.2 (GPB1)
- net GND: now also C1.2, C2.2, D7.4 (-)
- net IN1_1_L: now also U4.27 (GPA6); no longer U2.21 (GPA0)
- net IN1_2_L: now also U4.3 (GPB2); no longer U2.22 (GPA1)
- net IN2_1_L: now also U4.26 (GPA5); no longer U2.5 (GPB4)
- net IN2_2_L: now also U4.2 (GPB1); no longer U2.6 (GPB5)
- net IN3_1_L: now also U4.21 (GPA0); no longer U2.1 (GPB0)
- net IN3_2_L: now also U4.22 (GPA1); no longer U2.2 (GPB1)
- net IN4_1_L: now also U4.23 (GPA2); no longer U2.3 (GPB2)
- net IN4_2_L: now also U4.24 (GPA3); no longer U2.4 (GPB3)
- net LIGHT: now also U4.4 (GPB3); no longer U4.1 (GPB0)
- net M1_A: now also U4.1 (GPB0); no longer U2.7 (GPB6)
- net M2_A: now also U4.25 (GPA4); no longer U2.23 (GPA2)
- net REV1: now also U4.7 (GPB6); no longer U4.4 (GPB3)
- net REV2: now also U4.6 (GPB5); no longer U4.3 (GPB2)
- net SOUND: now also U4.28 (GPA7); no longer U4.6 (GPB5)
- net VBUS: now also C1.1, C2.1, D7.1 (+)
- net at K1.3, K2.3, U14.9 (Vin-): now also R1.2; no longer R2.2
- net at K3.3, K4.3, U3.9 (Vin-): now also R2.2; no longer R1.2
- no-connect marks 0 -> 2
Other:
- moved on the sheet: R1, R2

Commit message: update
Parts:
- added R27, R28, R29, R30: R0603_4.7k_1%_100mW_100PPM_AC, Resistor_SMD:R_0603_1608Metric, symbol Resistors_SMD_0603:R0603_4.7k_1%_100mW_100PPM_AC
Connections:
- net +3V3: now also U4.15 (A0), R27.1, R28.1
- net GND: now also U2.15 (A0), U2.16 (A1), U2.17 (A2), U4.16 (A1), U4.17 (A2)
- net GND2: now also MOD1.C1, MOD1.C3
- net IN3_1_L: now also U4.22 (GPA1); no longer U4.21 (GPA0)
- net IN3_2_L: now also U4.24 (GPA3); no longer U4.22 (GPA1)
- net IN4_1_L: now also U4.21 (GPA0); no longer U4.23 (GPA2)
- net IN4_2_L: now also U4.23 (GPA2); no longer U4.24 (GPA3)
- net SIG_CLOSE: now also MOD1.C2
- net SIG_OPEN: now also MOD1.C4
- net nSIG_CLOSE: now also R29.1; no longer U15.2
- net nSIG_OPEN: now also R30.1; no longer U1.2
- net at U4.18 (~{RESET}): now also R27.2
- net at U2.18 (~{RESET}): now also R28.2
- net at D7.2: now also MOD1.D11
- net at D7.3: now also MOD1.D12
- new net: R29.2, U15.2
- new net: R30.2, U1.2
Other:
- note added: "B00100000 0x20"
- note added: "B00100001 0x21"
- note added: "B01000000 0x40"
- note added: "B01000001 0x41"

Commit message: update
Parts:
- added U16: ESP32-DevKitC, PCM_Espressif:ESP32-DevKitC, symbol PCM_Espressif:ESP32-DevKitC
Connections:
- new net: U16.14 (GND), U16.32 (GND), U16.38 (GND)
Changed lines of the file:
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@@
 	(generator "eeschema")
 	(generator_version "8.0")
-	(paper "A3")
+	(paper "A2")
 	(junction
 		(at 281.94 129.54)
@@
 					(unit 1)
 				)
+			)
+		)
+	)
+	(symbol
+		(lib_id "PCM_Espressif:ESP32-DevKitC")
+		(at 99.06 344.17 0)
+		(unit 1)
+		(exclude_from_sim no)
+		(in_bom yes)
+		(on_board yes)
+		(dnp no)
+		(fields_autoplaced yes)
+		(property "Reference" "U16"
+			(at 101.2541 379.73 0)
+			(effects
+				(font
+					(size 1.27 1.27)
+				)
+				(justify left)
+			)
+		)
+		(property "Value" "ESP32-DevKitC"
+			(at 101.2541 382.27 0)
+			(effects
+				(font
+					(size 1.27 1.27)
+				)
+				(justify left)
+			)
+		)
+		(property "Footprint" "PCM_Espressif:ESP32-DevKitC"
+			(at 99.06 387.35 0)
+			(effects
+				(font
+					(size 1.27 1.27)
+				)
+				(hide yes)
+			)
+		)
+		(property "Datasheet" "https://docs.espressif.com/projects/esp-idf/zh_CN/latest/esp32/hw-reference/esp32/get-started-devkitc.html"
+			(at 99.06 389.89 0)
+			(effects
+				(font
+					(size 1.27 1.27)
+				)
+				(hide yes)
+			)
+		)
+		(property "Description" "Development Kit"
+			(at 99.06 344.17 0)
+			(effects
+				(font
+					(size 1.27 1.27)
+				)
+				(hide yes)
+			)
+		)
+		(pin "8"
+		)
+		(pin "38"
+		)
+		(pin "9"
+		)
+		(pin "5"
+		)
+		(pin "17"
+		)
+		(pin "26"
+		)
+		(pin "16"
+		)
+		(pin "25"
+		)
+		(pin "33"
+		)
+		(pin "21"
+		)
+		(pin "10"
+		)
+		(pin "24"
+		)
+		(pin "14"
+		)
+		(pin "13"
+		)
+		(pin "22"
+		)
+		(pin "23"
+		)
+		(pin "31"
+		)
+		(pin "3"
+		)
+		(pin "34"
+		)
+		(pin "2"
+		)
+		(pin "20"
+		)
+		(pin "29"
+		)
+		(pin "11"
+		)
+		(pin "6"
+		)
+		(pin "27"
+		)
+		(pin "15"
+		)
+		(pin "1"
+		)
+		(pin "32"
+		)
+		(pin "19"
+		)
+		(pin "18"
+		)
+		(pin "30"
+		)
+		(pin "36"
+		)
+		(pin "28"
+		)
+		(pin "37"
+		)
+		(pin "12"
+		)
+		(pin "7"
+		)
+		(pin "35"
+		)
+		(pin "4"
+		)
+		(instances
+			(project ""
+				(path "/369bf40f-e28a-46b1-be37-62b35f4960a2"
+					(reference "U16")
+					(unit 1)
+				)

Commit message: update
Parts:
- removed U16: ESP32-DevKitC, PCM_Espressif:ESP32-DevKitC, symbol PCM_Espressif:ESP32-DevKitC
- added R31, R32, R37, R38, R39, R40: R0603_4.7k_1%_100mW_100PPM_AC, Resistor_SMD:R_0603_1608Metric, symbol Resistors_SMD_0603:R0603_4.7k_1%_100mW_100PPM_AC
- added R33, R34, R35, R36: R0805_1.5k_1%_125mW_100PPM_AC, Resistor_SMD:R_0805_2012Metric, symbol Resistors_SMD_0805:R0805_1.5k_1%_125mW_100PPM_AC
- added U16, U17: LTV-817S, Package_DIP:SMDIP-4_W9.53mm, symbol Isolator:LTV-817S
Connections:
- net +3V3: now also MOD1.C12, R31.1, R32.1, R37.1, R38.1, R39.1, R40.1
- net GND: now also R34.1, R36.1, U16.3, U17.3
- net GND2: now also MOD1.C10
- net INT: now also R39.2
- net SCL: now also R38.2
- net SDA: now also R37.2
- net IN5_1_L: now reaches U2.1 (GPB0)
- net IN5_1_L: now also R32.2, U16.4
- net IN5_2_L: now reaches U2.2 (GPB1)
- net IN5_2_L: now also R31.2, U17.4
- net OWIRE: now reaches MOD1.C11
- net OWIRE: now also R40.2
- new net: R35.2, U17.1
- new net: R36.2, U17.2
- new net: R33.2, U16.1
- new net: R34.2, U16.2
- new net IN5_1_P: R33.1
- new net IN5_2_P: R35.1
Other:
- moved on the sheet: D1, D2, D3, D4, D5, D6, F2, J1, J2, K1, K2, K3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

Commit message: update
Parts:
- added D8, D9: SM4007, Diode_SMD:D_MELF, symbol Diode:SM4007
- added K7, K8: SANYOU_SRD_Form_C, Relay_THT:Relay_SPDT_SANYOU_SRD_Series_Form_C, symbol Relay:SANYOU_SRD_Form_C
Connections:
- net +24V: now also MOD1.D1, MOD1.D3, D8.1 (K), D9.1 (K), K7.2, K8.2
- net IN5_1_P: now also MOD1.D4
- net IN5_2_P: now also MOD1.D2
- net NC1: now reaches MOD1.D10
- net NC1: now also K7.4
- net NO2: now reaches MOD1.D5
- net NO2: now also K8.3
- net COM2: now reaches MOD1.D6
- net COM2: now also K8.1
- net NC2: now reaches MOD1.D7
- net NC2: now also K8.4
- net NO1: now reaches MOD1.D8
- net NO1: now also K7.3
- net COM1: now reaches MOD1.D9
- net COM1: now also K7.1
- new net nREL1: D8.2 (A), K7.5
- new net nREL2: D9.2 (A), K8.5

Commit message: update
Parts:
- added C3, C6: 100nF, Capacitor_THT:C_Disc_D5.0mm_W2.5mm_P5.00mm, symbol Device:C
- added C4, C5: 100uF, Capacitor_THT:CP_Radial_D8.0mm_P3.50mm, symbol Device:C_Polarized
- added J3, J4: Conn_01x05_Pin, Connector_JST:JST_EH_B6B-EH-A_1x06_P2.50mm_Vertical, symbol Connector:Conn_01x06_Pin
- added U18: R-78E3.3-1.0, Converter_DCDC:Converter_DCDC_RECOM_R-78E-0.5_THT, symbol Regulator_Switching:R-78E3.3-1.0
Connections:
- net +3V3: now also C3.1, C4.1, J3.1 (Pin_1), J4.1 (Pin_1), U18.3 (OUT)
- net GND: now also C3.2, C4.2, C5.2, C6.2, J3.5 (Pin_5), J4.5 (Pin_5), U18.2 (GND)
- net INT: now also J3.2 (Pin_2), J4.2 (Pin_2)
- net SCL: now also J3.4 (Pin_4), J4.4 (Pin_4)
- net SDA: now also J3.3 (Pin_3), J4.3 (Pin_3)
- net VBUS: now also C5.1, C6.1, J3.6 (Pin_6), J4.6 (Pin_6), U18.1 (IN)

Commit message: update
Parts:
- added C7, C8: 100nF, Capacitor_SMD:C_0603_1608Metric, symbol Device:C
- added JP1: Jumper_2_Bridged, Jumper:SolderJumper-2_P1.3mm_Open_RoundedPad1.0x1.5mm, symbol Jumper:Jumper_2_Bridged
Connections:
- net +24V: now also C5.1, C6.1, J3.6 (Pin_6), J4.6 (Pin_6), U18.1 (IN)
- net +3V3: now also C7.1, C8.1
- net GND: now also MOD1.C10, C7.2, C8.2, JP1.1 (A)
- net GND2: now also JP1.2 (B); no longer MOD1.C10
- net VBUS: no longer C5.1, C6.1, J3.6 (Pin_6), J4.6 (Pin_6), U18.1 (IN)
