File: pcb/ESPhome_greenhouse_controller.kicad_sch (KiCad schematic)
At the start: 90 parts, among them J1 Conn_01x04_Pin, J2 Conn_01x04_Pin, J3 Conn_01x05_Pin, J4 Conn_01x05_Pin, K1 SANYOU_SRD_Form_C, K2 SANYOU_SRD_Form_C, K3 SANYOU_SRD_Form_C, K4 SANYOU_SRD_Form_C, K5 SANYOU_SRD_Form_C, K6 SANYOU_SRD_Form_C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

Commit message: update
Connections:
- net nREL1: now also U5.16 (O1)
- net REL1: now reaches U5.1 (I1)
- net REL1: now also U2.3 (GPB2)
Changed lines of the file:
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@@
 	(wire
 		(pts
+			(xy 304.8 86.36) (xy 317.5 86.36)
+		)
+		(stroke
+			(width 0)
+			(type default)
+		)
+	)
+	(wire
+		(pts
 			(xy 304.8 191.77) (xy 317.5 191.77)
 		)
@@
 	(wire
 		(pts
+			(xy 461.01 227.33) (xy 473.71 227.33)
+		)
+		(stroke
+			(width 0)
+			(type default)
+		)
+	)
+	(wire
+		(pts
 			(xy 459.74 36.83) (xy 459.74 39.37)
 		)
@@
 	(wire
 		(pts
+			(xy 440.69 227.33) (xy 427.99 227.33)
+		)
+		(stroke
+			(width 0)
+			(type default)
+		)
+	)
+	(wire
+		(pts
 			(xy 459.74 142.24) (xy 459.74 143.51)
 		)
@@
 		)
 	)
+	(label "REL1"
+		(at 317.5 86.36 180)
+		(fields_autoplaced yes)
+		(effects
+			(font
+				(size 1.27 1.27)
+			)
+			(justify right bottom)
+		)
+	)
 	(label "nREV2"
 		(at 480.06 115.57 0)
@@
 		)
 	)
+	(label "nREL1"
+		(at 473.71 227.33 180)
+		(fields_autoplaced yes)
+		(effects
+			(font
+				(size 1.27 1.27)
+			)
+			(justify right bottom)
+		)
+	)
 	(label "SDA"
 		(at 454.66 172.72 90)
@@
 		)
 	)
+	(label "REL1"
+		(at 427.99 227.33 0)
+		(fields_autoplaced yes)
+		(effects
+			(font
+				(size 1.27 1.27)
+			)
+			(justify left bottom)
+		)
+	)

Commit message: update
Parts:
- added C10, C9: 100nF, Capacitor_SMD:C_0603_1608Metric, symbol Device:C
- added JP2: Jumper_2_Bridged, Jumper:SolderJumper-2_P1.3mm_Open_RoundedPad1.0x1.5mm, symbol Jumper:Jumper_2_Bridged
- added unit 5 of MOD1
Connections:
- net +24V: now also JP2.1 (A), MOD1.E1; no longer R1.1, R2.1, U14.10 (Vin+), U14.8 (Vbus), U3.10 (Vin+), U3.8 (Vbus)
- net +3V3: now also C10.1, C9.1
- net GND: now also C10.2, C9.2
- net nSIG_CLOSE: now also U2.5 (GPB4)
- net nSIG_OPEN: now also U2.6 (GPB5)
- net REL2: now reaches U2.4 (GPB3)
- new net MOTOR: JP2.2 (B), MOD1.E2, R1.1, R2.1, U14.10 (Vin+), U14.8 (Vbus), U3.10 (Vin+), U3.8 (Vbus)
Other:
- moved on the sheet: C8, F2

Commit message: update
Parts:
- added Q1: BC817, Package_TO_SOT_SMD:SOT-23, symbol Transistor_BJT:BC817
- U5: value ULN2003A -> ULN2803A; footprint Package_SO:SOIC-16W_5.3x10.2mm_P1.27mm -> Package_SO:SOIC-18W_7.5x11.6mm_P1.27mm; symbol Transistor_Array:ULN2003A -> Transistor_Array:ULN2803A
Connections:
- net +24V: now also U5.10 (COM); no longer U5.9 (COM)
- net FWD1: now also U5.7 (I7); no longer U5.6 (I6)
- net FWD2: now also U5.4 (I4); no longer U5.3 (I3)
- net GND: now also U5.9 (GND); no longer U5.8 (GND)
- net LIGHT: now also U5.3 (I3); no longer U5.2 (I2)
- net REL1: now also U5.2 (I2); no longer U5.1 (I1)
- net REV1: now also U5.6 (I6); no longer U5.5 (I5)
- net REV2: now also U5.5 (I5); no longer U5.4 (I4)
- net SOUND: now also U5.8 (I8); no longer U5.7 (I7)
- net nFWD1: now also U5.12 (O7); no longer U5.11 (O6)
- net nFWD2: now also U5.15 (O4); no longer U5.14 (O3)
- net nLIGHT: now also U5.16 (O3); no longer U5.15 (O2)
- net nREL1: now also U5.17 (O2); no longer U5.16 (O1)
- net nREV1: now also U5.13 (O6); no longer U5.12 (O5)
- net nREV2: now also U5.14 (O5); no longer U5.13 (O4)
- net nSOUND: now also U5.11 (O8); no longer U5.10 (O7)
Changed lines of the file:
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@@
+	)
+	(symbol
+		(lib_id "Transistor_BJT:BC817")
+		(at 449.58 316.23 0)
+		(unit 1)
+		(exclude_from_sim no)
+		(in_bom yes)
+		(on_board yes)
+		(dnp no)
+		(fields_autoplaced yes)
+		(property "Reference" "Q1"
+			(at 454.66 314.9599 0)
+			(effects
+				(font
+					(size 1.27 1.27)
+				)
+				(justify left)
+			)
+		)
+		(property "Value" "BC817"
+			(at 454.66 317.4999 0)
+			(effects
+				(font
+					(size 1.27 1.27)
+				)
+				(justify left)
+			)
+		)
+		(property "Footprint" "Package_TO_SOT_SMD:SOT-23"
+			(at 454.66 318.135 0)
+			(effects
+				(font
+					(size 1.27 1.27)
+					(italic yes)
+				)
+				(justify left)
+				(hide yes)
+			)
+		)
+		(property "Datasheet" "https://www.onsemi.com/pub/Collateral/BC818-D.pdf"
+			(at 449.58 316.23 0)
+			(effects
+				(font
+					(size 1.27 1.27)
+				)
+				(justify left)
+				(hide yes)
+			)
+		)
+		(property "Description" "0.8A Ic, 45V Vce, NPN Transistor, SOT-23"
+			(at 449.58 316.23 0)
+			(effects
+				(font
+					(size 1.27 1.27)
+				)
+				(hide yes)
+			)
+		)
+		(pin "1"
+		)
+		(pin "2"
+		)
+		(pin "3"
+		)
+		(instances
+			(project ""
+				(path "/369bf40f-e28a-46b1-be37-62b35f4960a2"
+					(reference "Q1")
+					(unit 1)
+				)
+			)
+		)
 	)
 	(symbol
@@
 	)
 	(symbol
-		(lib_id "Transistor_Array:ULN2003A")
-		(at 450.85 232.41 0)
+		(lib_id "Transistor_Array:ULN2803A")
+		(at 450.85 229.87 0)
 		(unit 1)
 		(exclude_from_sim no)
@@
 			)
 		)
-		(property "Value" "ULN2003A"
+		(property "Value" "ULN2803A"
 			(at 450.85 217.17 0)
 			(effects
@@
 			)
 		)
-		(property "Footprint" "Package_SO:SOIC-16W_5.3x10.2mm_P1.27mm"
+		(property "Footprint" "Package_SO:SOIC-18W_7.5x11.6mm_P1.27mm"
 			(at 452.12 246.38 0)
 			(effects
@@
 			)
 		)
-		(property "Datasheet" "http://www.ti.com/lit/ds/symlink/uln2003a.pdf"
-			(at 453.39 237.49 0)
-			(effects
-				(font
-					(size 1.27 1.27)
-				)
-				(hide yes)
-			)
-		)
-		(property "Description" "High Voltage, High Current Darlington Transistor Arrays, SOIC16/SOIC16W/DIP16/TSSOP16"
-			(at 450.85 232.41 0)
+		(property "Datasheet" "http://www.ti.com/lit/ds/symlink/uln2803a.pdf"
+			(at 453.39 234.95 0)
+			(effects
+				(font
+					(size 1.27 1.27)
+				)
+				(hide yes)
+			)
+		)
+		(property "Description" "Darlington Transistor Arrays, SOIC18/DIP18"
+			(at 450.85 229.87 0)
 			(effects
 				(font
@@
 		(pin "16"
 		)
-		(instances
+		(pin "18"
+		)
+		(pin "17"
+		)
+		(instances

Commit message: update
Parts:
- removed C5: 100uF, Capacitor_THT:CP_Radial_D8.0mm_P3.50mm, symbol Device:C_Polarized
- removed J1, J2: Conn_01x04_Pin, symbol 380-015-113L001:Conn_01x04_Pin
- added J1: Conn_01x05_Pin, Connector_PinHeader_2.54mm:PinHeader_1x05_P2.54mm_Vertical, symbol Connector:Conn_01x05_Pin
- C3, C6: footprint Capacitor_THT:C_Disc_D5.0mm_W2.5mm_P5.00mm -> Capacitor_SMD:C_0805_2012Metric
Connections:
- net REL2: now also U5.1 (I1)
- net nREL2: now also U5.18 (O1)
- net 1: now reaches U2.21 (GPA0)
- net 1: now also MOD1.C5
- net 2: now reaches U2.22 (GPA1)
- net 2: now also MOD1.C6
- net 3: now reaches U2.23 (GPA2)
- net 3: now also MOD1.C7
- net 4: now reaches U2.24 (GPA3)
- net 4: now also MOD1.C8
- net 5: now reaches U2.25 (GPA4)
- net 5: now also MOD1.C9
- net 6: now reaches U2.26 (GPA5)
- net 6: now also J1.2 (Pin_2)
- net 7: now reaches U2.27 (GPA6)
- net 7: now also J1.3 (Pin_3)
- net 8: now reaches U2.7 (GPB6)
- net 8: now also J1.4 (Pin_4)
Other:
- moved on the sheet: JP1, MOD1C
