File: pcb/ESPhome_greenhouse_controller.kicad_pcb (KiCad board)
At the start: 2 copper layers, 15 parts, among them K1 SANYOU_SRD_Form_C, K2 SANYOU_SRD_Form_C, K3 SANYOU_SRD_Form_C, K4 SANYOU_SRD_Form_C, K5 SANYOU_SRD_Form_C, K6 SANYOU_SRD_Form_C, U1 PC817, U2 PC817, U3 INA219AxD, U4 INA219AxD

Commit message: update
Parts:
- added D3: SM4007, Diode_SMD:D_MELF, F.Cu at (190.5, 48.4)
- added D4: SM4007, Diode_SMD:D_MELF, F.Cu at (190.5, 52.7)
- added D5: SM4007, Diode_SMD:D_MELF, F.Cu at (190.5, 57.1)
- added D6: SM4007, Diode_SMD:D_MELF, F.Cu at (190.5, 61.4)
- U1, U2: value PC817 -> EL817

Commit message: update
Parts:
- added MOD1: ~, kadex:ZD1008, F.Cu at (81.4, 110.0)
- moved K1 113.8 mm to (181.9, 118.5), turned to -90 degrees
- moved K2 90.3 mm to (165.4, 118.5), turned to -90 degrees
- moved K3 66.7 mm to (148.7, 118.5), turned to -90 degrees
- moved K4 43.2 mm to (131.8, 118.5), turned to -90 degrees
- moved K5 21.1 mm to (115.0, 118.5), turned to -90 degrees
- moved K6 11.9 mm to (98.7, 118.5), turned to -90 degrees
Other:
- board outline added: 135.7 x 83 mm

Commit message: update
Parts:
- added R10: R0603_4.7k_1%_100mW_100PPM_AC, Resistor_SMD:R_0603_1608Metric, F.Cu at (46.2, 71.5)
- added R11: R0805_1.5k_1%_125mW_100PPM_AC, Resistor_SMD:R_0805_2012Metric, B.Cu at (99.0, 132.2)
- added R12: R0805_1.5k_1%_125mW_100PPM_AC, Resistor_SMD:R_0805_2012Metric, B.Cu at (96.7, 132.2)
- added R13: R0805_1.5k_1%_125mW_100PPM_AC, Resistor_SMD:R_0805_2012Metric, B.Cu at (103.8, 132.3)
- added R14: R0805_1.5k_1%_125mW_100PPM_AC, Resistor_SMD:R_0805_2012Metric, B.Cu at (101.3, 132.3)
- added R15: R0603_4.7k_1%_100mW_100PPM_AC, Resistor_SMD:R_0603_1608Metric, F.Cu at (249.8, 120.8)
- added R16: R0603_4.7k_1%_100mW_100PPM_AC, Resistor_SMD:R_0603_1608Metric, F.Cu at (249.8, 123.3)
- added R17: R0805_1.5k_1%_125mW_100PPM_AC, Resistor_SMD:R_0805_2012Metric, F.Cu at (245.6, 121.0)
- added R18: R0805_1.5k_1%_125mW_100PPM_AC, Resistor_SMD:R_0805_2012Metric, F.Cu at (245.6, 124.0)
- added R19: R0805_1.5k_1%_125mW_100PPM_AC, Resistor_SMD:R_0805_2012Metric, F.Cu at (245.6, 127.0)
- added R20: R0805_1.5k_1%_125mW_100PPM_AC, Resistor_SMD:R_0805_2012Metric, F.Cu at (245.6, 129.9)
- added R21: R0603_4.7k_1%_100mW_100PPM_AC, Resistor_SMD:R_0603_1608Metric, F.Cu at (249.8, 125.8)
- added R22: R0603_4.7k_1%_100mW_100PPM_AC, Resistor_SMD:R_0603_1608Metric, F.Cu at (249.8, 128.4)
- added R23: R0805_1.5k_1%_125mW_100PPM_AC, Resistor_SMD:R_0805_2012Metric, F.Cu at (245.6, 132.8)
- added R24: R0805_1.5k_1%_125mW_100PPM_AC, Resistor_SMD:R_0805_2012Metric, F.Cu at (245.6, 135.8)
- added R25: R0805_1.5k_1%_125mW_100PPM_AC, Resistor_SMD:R_0805_2012Metric, F.Cu at (245.6, 138.8)
- added R26: R0805_1.5k_1%_125mW_100PPM_AC, Resistor_SMD:R_0805_2012Metric, F.Cu at (245.6, 141.7)
- added R3: R0603_4.7k_1%_100mW_100PPM_AC, Resistor_SMD:R_0603_1608Metric, F.Cu at (65.7, 108.5)
- added R4: R0603_4.7k_1%_100mW_100PPM_AC, Resistor_SMD:R_0603_1608Metric, F.Cu at (65.7, 111.0)
- added R5: R0805_1.5k_1%_125mW_100PPM_AC, Resistor_SMD:R_0805_2012Metric, F.Cu at (96.7, 132.2)
- added R6: R0805_1.5k_1%_125mW_100PPM_AC, Resistor_SMD:R_0805_2012Metric, F.Cu at (99.0, 132.2)
- added R7: R0805_1.5k_1%_125mW_100PPM_AC, Resistor_SMD:R_0805_2012Metric, F.Cu at (101.3, 132.3)
- added R8: R0805_1.5k_1%_125mW_100PPM_AC, Resistor_SMD:R_0805_2012Metric, F.Cu at (103.8, 132.3)
- added R9: R0603_4.7k_1%_100mW_100PPM_AC, Resistor_SMD:R_0603_1608Metric, F.Cu at (46.2, 69.0)
- added U10: LTV-817S, Package_DIP:SMDIP-4_W9.53mm, F.Cu at (236.8, 122.9)
- added U11: LTV-817S, Package_DIP:SMDIP-4_W9.53mm, F.Cu at (236.8, 129.6)
- added U12: LTV-817S, Package_DIP:SMDIP-4_W9.53mm, F.Cu at (236.8, 136.2)
- added U13: LTV-817S, Package_DIP:SMDIP-4_W9.53mm, F.Cu at (207.7, 124.1)
- added U14: STM32F103CBTx, Package_QFP:LQFP-48_7x7mm_P0.5mm, F.Cu at (155.0, 109.0)
- added U5: ULN2003A, Package_SO:SOIC-16W_5.3x10.2mm_P1.27mm, F.Cu at (114.0, 112.8)
- added U6: LTV-817S, Package_DIP:SMDIP-4_W9.53mm, F.Cu at (96.7, 123.9)
- added U7: LTV-817S, Package_DIP:SMDIP-4_W9.53mm, F.Cu at (102.5, 124.0)
- added U8: LTV-817S, Package_DIP:SMDIP-4_W9.53mm, B.Cu at (96.7, 123.9)
- added U9: LTV-817S, Package_DIP:SMDIP-4_W9.53mm, B.Cu at (102.5, 124.0)
- D1, D2, D3, D4, D5, D6, R1, R2, U3, U4: moved to B.Cu
- moved D2 113.9 mm to (138.4, 137.7)
- moved D5 107.2 mm to (114.2, 132.3), turned to 180 degrees
- moved D1 102.8 mm to (124.3, 129.6), turned to -90 degrees
- moved K6 99.4 mm to (196.4, 136.5), turned to 90 degrees
- moved D3 96.1 mm to (154.9, 137.7)
- moved D4 87.0 mm to (171.7, 137.7)
- moved MOD1 73.7 mm to (155.1, 110.0)
- moved D6 68.2 mm to (190.9, 129.6), turned to -90 degrees
- moved F2 63.4 mm to (91.2, 103.7), turned to -90 degrees
- moved U1 59.9 mm to (128.8, 47.9)
- moved U2 59.9 mm to (128.8, 54.6)
- moved R1 56.6 mm to (132.2, 122.3)
- moved K1 54.7 mm to (130.2, 136.4), turned to 90 degrees
- moved K4 51.4 mm to (179.9, 136.5), turned to 90 degrees
- moved R2 49.3 mm to (165.2, 122.3)
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Connections:
- K1 pad 3: Net-(U3-IN+) -> Net-(U3-IN-)
- K1 pad 4: GND1 -> GND
- K1 pad 5: /nFWD1 -> /nREV1
- K2 pad 3: Net-(U3-IN+) -> Net-(U3-IN-)
- K2 pad 4: GND1 -> GND
- K2 pad 5: /nREV1 -> /nFWD1
- K3 pad 3: Net-(U4-IN+) -> Net-(U4-IN-)
- K3 pad 4: GND1 -> GND
- K4 pad 3: Net-(U4-IN+) -> Net-(U4-IN-)
- K4 pad 4: GND1 -> GND
- K5 pad 1: /SOUND -> /SOUND+
- K6 pad 1: /LIGHT -> /LIGHT+
- MOD1 pad A1: unconnected-(MOD1-PadA1) -> +24V
- MOD1 pad A10: (no net) -> GND
- MOD1 pad A11: (no net) -> /M1+
- MOD1 pad A12: (no net) -> /M1-
- MOD1 pad A2: unconnected-(MOD1-PadA2) -> /IN1_1_P
- MOD1 pad A3: unconnected-(MOD1-PadA3) -> +24V
- MOD1 pad A4: unconnected-(MOD1-PadA4) -> /IN1_2_P
- MOD1 pad A5: unconnected-(MOD1-PadA5) -> +24V
- MOD1 pad A6: unconnected-(MOD1-PadA6) -> /IN2_1_P
- MOD1 pad A7: unconnected-(MOD1-PadA7) -> +24V
- MOD1 pad A8: unconnected-(MOD1-PadA8) -> /IN2_2_P
- MOD1 pad A9: (no net) -> /SOUND+
- R1 pad 2: Net-(U3-IN+) -> Net-(U3-IN-)
- R2 pad 2: Net-(U4-IN+) -> Net-(U4-IN-)
- U3 pad 7: +24V -> Net-(U3-IN-)
- U3 pad 8: Net-(U3-IN+) -> +24V
- U4 pad 7: +24V -> Net-(U4-IN-)
- U4 pad 8: Net-(U4-IN+) -> +24V
Routing:
- net +24V: track 0.00 -> 242.1 mm
- net GND: track 0.00 -> 131.8 mm
- net /nLIGHT: track 0.00 -> 89.1 mm, vias 0 -> 2
- net /nFWD2: track 0.00 -> 74.7 mm
- net /nREV2: track 0.00 -> 60.1 mm
- net /nFWD1: track 0.00 -> 45.0 mm
- net Net-(U4-IN-): track 0.00 -> 31.8 mm
- net /IN2_2_P: track 0.00 -> 31.4 mm
- net /nREV1: track 0.00 -> 29.4 mm
- net /IN2_1_P: track 0.00 -> 25.9 mm
- net Net-(U3-IN-): track 0.00 -> 25.5 mm
- net /nSOUND: track 0.00 -> 24.7 mm
- net /SOUND+: track 0.00 -> 22.8 mm
- net /LIGHT+: track 0.00 -> 22.6 mm
- net /M1+: track 0.00 -> 15.8 mm
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- added copper zone on B.Cu, net +24V

Commit message: update
Parts:
- removed U2: EL817, Package_DIP:DIP-4_W7.62mm
- added U15: LTV-817S, Package_DIP:SMDIP-4_W9.53mm, F.Cu at (248.7, 103.7)
- R21, R22, R23, R24, R25, R26, U12, U13: moved to B.Cu
- U1: value EL817 -> LTV-817S; footprint Package_DIP:DIP-4_W7.62mm -> Package_DIP:SMDIP-4_W9.53mm
- moved U1 129.6 mm to (248.7, 97.1)
- moved R16 42.6 mm to (207.8, 116.4), turned to 180 degrees
- moved R22 41.6 mm to (210.0, 116.4), turned to 180 degrees
- moved R26 40.4 mm to (206.2, 132.5), turned to 90 degrees
- moved R19 39.7 mm to (206.3, 132.5), turned to 90 degrees
- moved R15 39.2 mm to (210.9, 116.4)
- moved R21 37.9 mm to (213.1, 116.4)
- moved R25 37.4 mm to (208.8, 132.5), turned to 90 degrees
- moved R20 36.9 mm to (208.8, 132.5), turned to 90 degrees
- moved R17 35.9 mm to (211.6, 132.5), turned to 90 degrees
- moved R24 34.1 mm to (211.6, 132.5), turned to 90 degrees
- moved R18 32.8 mm to (213.9, 132.5), turned to 90 degrees
- moved R23 31.7 mm to (213.9, 132.5), turned to 90 degrees
- moved U11 29.6 mm to (207.7, 124.1), turned to 90 degrees
- moved U12 26.3 mm to (213.5, 124.1), turned to 90 degrees
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Connections:
- MOD1 pad B10: unconnected-(MOD1-PadB10) -> +24V
- MOD1 pad B11: unconnected-(MOD1-PadB11) -> /IN3_1_P
- MOD1 pad B12: unconnected-(MOD1-PadB12) -> +24V
- MOD1 pad B5: unconnected-(MOD1-PadB5) -> /IN4_2_P
- MOD1 pad B6: unconnected-(MOD1-PadB6) -> +24V
- MOD1 pad B7: unconnected-(MOD1-PadB7) -> /IN4_1_P
- MOD1 pad B8: unconnected-(MOD1-PadB8) -> +24V
- MOD1 pad B9: unconnected-(MOD1-PadB9) -> /IN3_2_P
- U1 pad 2: /nSIG_CLOSE -> /nSIG_OPEN
- U1 pad 4: /SIG_CLOSE -> /SIG_OPEN
- U14 pad 1: unconnected-(U14-VBAT-Pad1) -> +3V3
- U14 pad 23: Net-(U14-VSS-Pad23) -> GND
- U14 pad 24: unconnected-(U14-VDD-Pad24) -> +3V3
- U14 pad 35: Net-(U14-VSS-Pad23) -> GND
- U14 pad 36: unconnected-(U14-VDD-Pad36) -> +3V3
- U14 pad 47: Net-(U14-VSS-Pad23) -> GND
- U14 pad 48: unconnected-(U14-VDD-Pad48) -> +3V3
- U14 pad 8: unconnected-(U14-VSSA-Pad8) -> GND
- U14 pad 9: unconnected-(U14-VDDA-Pad9) -> +3V3
Routing:
- net +24V: track 242.1 -> 302.6 mm
- net /SCL: track 0.00 -> 37.8 mm, vias 0 -> 2
- net /SDA: track 0.00 -> 36.8 mm
- net /IN4_2_P: track 0.00 -> 33.4 mm
- net /IN4_1_P: track 0.00 -> 28.9 mm
- net /IN3_2_P: track 0.00 -> 13.0 mm
- net /IN3_1_P: track 0.00 -> 12.0 mm
- net Net-(U3-IN-): track 25.5 -> 32.3 mm
- net /nREV1: track 29.4 -> 30.1 mm

Commit message: update
Parts:
- added R27: R0603_10k_1%_100mW_100PPM_AC, Resistor_SMD:R_0603_1608Metric, F.Cu at (55.4, 126.6)
- added U2: MCP23017_SO, Package_SO:SOIC-28W_7.5x17.9mm_P1.27mm, F.Cu at (135.8, 101.3)
- moved U1 44.8 mm to (204.9, 87.6), turned to 90 degrees
- moved U15 40.5 mm to (211.6, 87.6), turned to 90 degrees
Connections:
- R10 pad 1: P-UP -> +3V3
- R10 pad 2: /IN2_L -> /IN2_2_L
- R15 pad 1: P-UP -> +3V3
- R16 pad 1: P-UP -> +3V3
- R21 pad 1: P-UP -> +3V3
- R21 pad 2: /IN1_L -> /IN4_1_L
- R22 pad 1: P-UP -> +3V3
- R22 pad 2: /IN2_L -> /IN4_2_L
- R3 pad 1: P-UP -> +3V3
- R3 pad 2: /IN1_L -> /IN1_1_L
- R4 pad 1: P-UP -> +3V3
- R4 pad 2: /IN2_L -> /IN1_2_L
- R9 pad 1: P-UP -> +3V3
- R9 pad 2: /IN1_L -> /IN2_1_L
- U12 pad 4: /IN1_L -> /IN4_1_L
- U13 pad 4: /IN2_L -> /IN4_2_L
- U14 pad 18: unconnected-(U14-PB0-Pad18) -> /IN3_1_L
- U14 pad 19: unconnected-(U14-PB1-Pad19) -> /IN3_2_L
- U14 pad 20: unconnected-(U14-PB2-Pad20) -> /IN4_1_L
- U14 pad 30: unconnected-(U14-PA9-Pad30) -> /TX
- U14 pad 31: unconnected-(U14-PA10-Pad31) -> /RX
- U14 pad 34: unconnected-(U14-PA13-Pad34) -> /SWDIO
- U14 pad 37: unconnected-(U14-PA14-Pad37) -> /SWCLK
- U14 pad 39: unconnected-(U14-PB3-Pad39) -> /IN4_2_L
- U14 pad 40: unconnected-(U14-PB4-Pad40) -> /IN2_1_L
- U14 pad 41: unconnected-(U14-PB5-Pad41) -> /IN2_2_L
- U14 pad 42: unconnected-(U14-PB6-Pad42) -> /SCL
- U14 pad 43: unconnected-(U14-PB7-Pad43) -> /SDA
- U14 pad 44: unconnected-(U14-BOOT0-Pad44) -> /BOOT0
- U14 pad 45: unconnected-(U14-PB8-Pad45) -> /IN1_1_L
- U14 pad 46: unconnected-(U14-PB9-Pad46) -> /IN1_2_L
- U14 pad 7: unconnected-(U14-NRST-Pad7) -> /NRST
- U6 pad 4: /IN1_L -> /IN1_1_L
- U7 pad 4: /IN2_L -> /IN1_2_L
- U8 pad 4: /IN1_L -> /IN2_1_L
- U9 pad 4: /IN2_L -> /IN2_2_L

Commit message: update
Parts:
- removed U4: INA219AxD, Package_SO:SOIC-8_3.9x4.9mm_P1.27mm
- U14: value STM32F103CBTx -> INA237; footprint Package_QFP:LQFP-48_7x7mm_P0.5mm -> Package_SO:VSSOP-10_3x3mm_P0.5mm; moved to B.Cu
- U3: value INA219AxD -> INA237; footprint Package_SO:SOIC-8_3.9x4.9mm_P1.27mm -> Package_SO:VSSOP-10_3x3mm_P0.5mm
- moved U2 16.3 mm to (152.0, 103.6)
- moved U14 13.4 mm to (165.4, 114.2), turned to -90 degrees
Connections:
- D1 pad 2: /nREV1 -> /nFWD1
- D2 pad 2: /nFWD1 -> /nREV1
- K1 pad 3: Net-(U3-IN-) -> Net-(U14-Vin-)
- K1 pad 5: /nREV1 -> /nFWD1
- K2 pad 3: Net-(U3-IN-) -> Net-(U14-Vin-)
- K2 pad 5: /nFWD1 -> /nREV1
- K3 pad 3: Net-(U4-IN-) -> Net-(U3-Vin-)
- K4 pad 3: Net-(U4-IN-) -> Net-(U3-Vin-)
- R1 pad 2: Net-(U3-IN-) -> Net-(U14-Vin-)
- R2 pad 2: Net-(U4-IN-) -> Net-(U3-Vin-)
- U14 pad 1: +3V3 -> GND
- U14 pad 10: unconnected-(U14-PA0-Pad10) -> +24V
- U14 pad 2: unconnected-(U14-PC13-Pad2) -> GND
- U14 pad 3: unconnected-(U14-PC14-Pad3) -> /M1_A
- U14 pad 4: unconnected-(U14-PC15-Pad4) -> /SDA
- U14 pad 5: unconnected-(U14-PD0-Pad5) -> /SCL
- U14 pad 6: unconnected-(U14-PD1-Pad6) -> +3V3
- U14 pad 7: /NRST -> GND
- U14 pad 8: GND -> +24V
- U14 pad 9: +3V3 -> Net-(U14-Vin-)
- U2 pad 1: unconnected-(U2-GPB0-Pad1) -> /IN3_1_L
- U2 pad 10: unconnected-(U2-VSS-Pad10) -> GND
- U2 pad 12: unconnected-(U2-SCK-Pad12) -> /SCL
- U2 pad 13: unconnected-(U2-SDA-Pad13) -> /SDA
- U2 pad 2: unconnected-(U2-GPB1-Pad2) -> /IN3_2_L
- U2 pad 21: unconnected-(U2-GPA0-Pad21) -> /IN1_1_L
- U2 pad 22: unconnected-(U2-GPA1-Pad22) -> /IN1_2_L
- U2 pad 3: unconnected-(U2-GPB2-Pad3) -> /IN4_1_L
- U2 pad 4: unconnected-(U2-GPB3-Pad4) -> /IN4_2_L
- U2 pad 5: unconnected-(U2-GPB4-Pad5) -> /IN2_1_L
- U2 pad 6: unconnected-(U2-GPB5-Pad6) -> /IN2_2_L
- U2 pad 9: unconnected-(U2-VDD-Pad9) -> +3V3
- U3 pad 2: GND -> +3V3
- U3 pad 3: /SDA -> /M2_A
- U3 pad 4: /SCL -> /SDA
- U3 pad 5: +3V3 -> /SCL
- U3 pad 6: GND -> +3V3
- U3 pad 7: Net-(U3-IN-) -> GND
- U5 pad 11: /nREV1 -> /nFWD1
- U5 pad 12: /nFWD1 -> /nREV1
Routing:
- net Net-(U4-IN-): track 31.9 -> 0.00 mm
- net Net-(U3-Vin-): track 0.00 -> 31.9 mm
- net /nREV1: track 30.1 -> 45.0 mm
- net /nFWD1: track 45.0 -> 30.1 mm

Commit message: update
Parts:
- added U4: MCP23017_SO, Package_SO:SOIC-28W_7.5x17.9mm_P1.27mm, F.Cu at (180.3, 103.2)
Connections:
- U2 pad 23: unconnected-(U2-GPA2-Pad23) -> /M2_A
- U2 pad 7: unconnected-(U2-GPB6-Pad7) -> /M1_A
- U5 pad 2: unconnected-(U5-I2-Pad2) -> /LIGHT
- U5 pad 3: unconnected-(U5-I3-Pad3) -> /FWD2
- U5 pad 4: unconnected-(U5-I4-Pad4) -> /REV2
- U5 pad 5: unconnected-(U5-I5-Pad5) -> /REV1
- U5 pad 6: unconnected-(U5-I6-Pad6) -> /FWD1
- U5 pad 7: unconnected-(U5-I7-Pad7) -> /SOUND
Routing:
- net Net-(U3-IN-): track 32.3 -> 0.00 mm
- net (no net): track 0.00 -> 32.3 mm

Commit message: update
Parts:
- removed R27: R0603_10k_1%_100mW_100PPM_AC, Resistor_SMD:R_0603_1608Metric
- moved R10 71.2 mm to (105.1, 111.4)
- moved R9 67.9 mm to (99.2, 111.4)
- moved R4 36.5 mm to (102.2, 111.4), turned to 180 degrees
- moved R2 33.1 mm to (132.2, 122.3)
- moved R1 33.0 mm to (165.1, 122.4)
- moved R3 30.7 mm to (96.2, 111.4), turned to 180 degrees
- moved R16 1.59 mm to (206.4, 115.6), turned to 90 degrees
- moved U3 0.30 mm to (133.4, 113.7)
- moved U14 0.20 mm to (165.4, 114.0)
Connections:
- R1 pad 2: Net-(U14-Vin-) -> Net-(U3-Vin-)
- R2 pad 2: Net-(U3-Vin-) -> Net-(U14-Vin-)
Routing:
- net GND: track 131.8 -> 236.6 mm, vias 0 -> 9
- net (no net): track 32.3 -> 0.00 mm
- net +24V: track 302.6 -> 289.1 mm
- net Net-(U3-Vin-): track 31.9 -> 22.6 mm
- net /IN2_2_L: track 0.00 -> 8.73 mm, vias 0 -> 1
- net /IN2_1_L: track 0.00 -> 8.61 mm, vias 0 -> 1
- net /IN1_1_L: track 0.00 -> 8.03 mm
- net /IN1_2_L: track 0.00 -> 7.90 mm
- net Net-(R23-Pad2): track 0.00 -> 3.08 mm
- net Net-(R18-Pad2): track 0.00 -> 3.08 mm
- net Net-(R24-Pad2): track 0.00 -> 2.98 mm
- net Net-(R17-Pad2): track 0.00 -> 2.98 mm
- net Net-(R25-Pad2): track 0.00 -> 2.81 mm
- net Net-(R26-Pad2): track 0.00 -> 2.80 mm
- net Net-(R20-Pad2): track 0.00 -> 2.75 mm
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