File: pcb/ESPhome_greenhouse_controller.kicad_pcb (KiCad board)
At the start: 2 copper layers, 135.7 x 83 mm, 55 parts, among them K1 SANYOU_SRD_Form_C, K2 SANYOU_SRD_Form_C, K3 SANYOU_SRD_Form_C, K4 SANYOU_SRD_Form_C, K5 SANYOU_SRD_Form_C, K6 SANYOU_SRD_Form_C, U1 LTV-817S, U10 LTV-817S, U11 LTV-817S, U12 LTV-817S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

Commit message: update
Parts:
- added C1: EKM227M1HG1BRRSHP, Capacitor_THT:CP_Radial_D10.0mm_P5.00mm, F.Cu at (96.0, 111.3)
- added C2: EKM227M1HG1BRRSHP, Capacitor_THT:CP_Radial_D10.0mm_P5.00mm, F.Cu at (96.0, 100.7)
- added D7: GBU6D, Diode_THT:Diode_Bridge_Vishay_GBU, F.Cu at (90.0, 107.4)
- moved U2 103.0 mm to (254.9, 108.5)
- moved R1 32.9 mm to (132.2, 122.4)
- moved R2 32.8 mm to (165.0, 122.3)
- moved U4 32.4 mm to (148.8, 110.5)
- moved U14 32.0 mm to (133.4, 113.9)
- moved U3 32.0 mm to (165.4, 113.7)
- moved F2 13.2 mm to (90.8, 116.8)
- moved R3 6.05 mm to (95.2, 117.4)
- moved R4 6.05 mm to (101.2, 117.4)
- moved R9 6.05 mm to (98.2, 117.4)
- moved R10 6.05 mm to (104.1, 117.4)
- moved R12 1.80 mm to (96.7, 134.0)
- moved R13 1.80 mm to (103.8, 134.1)
- moved R14 1.80 mm to (101.3, 134.1)
- moved R5 1.80 mm to (96.7, 134.0)
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Connections:
- R1 pad 2: Net-(U3-Vin-) -> Net-(U14-Vin-)
- R2 pad 2: Net-(U14-Vin-) -> Net-(U3-Vin-)
- U2 pad 1: /IN3_1_L -> unconnected-(U2-GPB0-Pad1)
- U2 pad 19: unconnected-(U2-INTB-Pad19) -> /INT
- U2 pad 2: /IN3_2_L -> unconnected-(U2-GPB1-Pad2)
- U2 pad 20: unconnected-(U2-INTA-Pad20) -> /INT
- U2 pad 21: /IN1_1_L -> unconnected-(U2-GPA0-Pad21)
- U2 pad 22: /IN1_2_L -> unconnected-(U2-GPA1-Pad22)
- U2 pad 23: /M2_A -> unconnected-(U2-GPA2-Pad23)
- U2 pad 3: /IN4_1_L -> unconnected-(U2-GPB2-Pad3)
- U2 pad 4: /IN4_2_L -> unconnected-(U2-GPB3-Pad4)
- U2 pad 5: /IN2_1_L -> unconnected-(U2-GPB4-Pad5)
- U2 pad 6: /IN2_2_L -> unconnected-(U2-GPB5-Pad6)
- U2 pad 7: /M1_A -> unconnected-(U2-GPB6-Pad7)
- U4 pad 1: /LIGHT -> /M1_A
- U4 pad 19: unconnected-(U4-INTB-Pad19) -> /INT
- U4 pad 2: /FWD2 -> /IN2_2_L
- U4 pad 20: unconnected-(U4-INTA-Pad20) -> /INT
- U4 pad 21: unconnected-(U4-GPA0-Pad21) -> /IN3_1_L
- U4 pad 22: unconnected-(U4-GPA1-Pad22) -> /IN3_2_L
- U4 pad 23: unconnected-(U4-GPA2-Pad23) -> /IN4_1_L
- U4 pad 24: unconnected-(U4-GPA3-Pad24) -> /IN4_2_L
- U4 pad 25: unconnected-(U4-GPA4-Pad25) -> /M2_A
- U4 pad 26: unconnected-(U4-GPA5-Pad26) -> /IN2_1_L
- U4 pad 27: unconnected-(U4-GPA6-Pad27) -> /IN1_1_L
- U4 pad 28: unconnected-(U4-GPA7-Pad28) -> /SOUND
- U4 pad 3: /REV2 -> /IN1_2_L
- U4 pad 4: /REV1 -> /LIGHT
- U4 pad 5: /FWD1 -> /FWD2
- U4 pad 6: /SOUND -> /REV2
- U4 pad 7: unconnected-(U4-GPB6-Pad7) -> /REV1
- U4 pad 8: unconnected-(U4-GPB7-Pad8) -> /FWD1
Routing:
- net +3V3: track 0.00 -> 65.2 mm, vias 0 -> 5
- net GND: track 236.6 -> 297.5 mm, vias 9 -> 10
- net /IN1_1_L: track 8.03 -> 62.3 mm
- net /IN1_2_L: track 7.90 -> 59.5 mm
- net /IN2_1_L: track 8.61 -> 58.9 mm
- net /IN2_2_L: track 8.73 -> 54.5 mm
- net /FWD1: track 0.00 -> 45.2 mm
- net /REV1: track 0.00 -> 42.2 mm
- net /REV2: track 0.00 -> 39.2 mm
- net /SOUND: track 0.00 -> 36.7 mm, vias 0 -> 2
- net +24V: track 289.1 -> 325.2 mm, vias 0 -> 1
- net /FWD2: track 0.00 -> 36.0 mm
- net /LIGHT: track 0.00 -> 32.8 mm
- net VBUS: track 0.00 -> 30.2 mm
- net unconnected-(D7-Pad2): track 0.00 -> 27.6 mm
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
Commit message: update
Parts:
- added R27: R0603_4.7k_1%_100mW_100PPM_AC, Resistor_SMD:R_0603_1608Metric, F.Cu at (154.1, 103.7)
- added R28: R0603_4.7k_1%_100mW_100PPM_AC, Resistor_SMD:R_0603_1608Metric, F.Cu at (233.2, 104.8)
- added R29: R0603_4.7k_1%_100mW_100PPM_AC, Resistor_SMD:R_0603_1608Metric, F.Cu at (210.1, 94.2)
- added R30: R0603_4.7k_1%_100mW_100PPM_AC, Resistor_SMD:R_0603_1608Metric, F.Cu at (210.1, 96.7)
- R21, R22: moved to F.Cu
- moved R21 2.06 mm to (215.2, 116.2)
- moved R15 1.23 mm to (212.1, 116.2), turned to 180 degrees
- moved R22 0.96 mm to (209.1, 116.2), turned to 0 degrees
- moved U1 0.95 mm to (205.8, 87.6)
- moved R16 0.76 mm to (206.0, 116.2), turned to 180 degrees
Connections:
- D7 pad 2: unconnected-(D7-Pad2) -> Net-(D7-Pad2)
- D7 pad 3: unconnected-(D7-Pad3) -> Net-(D7-Pad3)
- MOD1 pad C1: unconnected-(MOD1-PadC1) -> GND2
- MOD1 pad C10: (no net) -> unconnected-(MOD1-PadC10)
- MOD1 pad C11: (no net) -> unconnected-(MOD1-PadC11)
- MOD1 pad C12: (no net) -> unconnected-(MOD1-PadC12)
- MOD1 pad C2: unconnected-(MOD1-PadC2) -> /SIG_CLOSE
- MOD1 pad C3: unconnected-(MOD1-PadC3) -> GND2
- MOD1 pad C4: unconnected-(MOD1-PadC4) -> /SIG_OPEN
- MOD1 pad C9: (no net) -> unconnected-(MOD1-PadC9)
- MOD1 pad D10: (no net) -> unconnected-(MOD1-PadD10)
- MOD1 pad D11: (no net) -> Net-(D7-Pad2)
- MOD1 pad D12: (no net) -> Net-(D7-Pad3)
- MOD1 pad D9: (no net) -> unconnected-(MOD1-PadD9)
- U1 pad 2: /nSIG_OPEN -> Net-(R30-Pad2)
- U15 pad 2: /nSIG_CLOSE -> Net-(R29-Pad2)
- U2 pad 15: unconnected-(U2-A0-Pad15) -> GND
- U2 pad 16: unconnected-(U2-A1-Pad16) -> GND
- U2 pad 17: unconnected-(U2-A2-Pad17) -> GND
- U2 pad 18: unconnected-(U2-~{RESET}-Pad18) -> Net-(U2-~{RESET})
- U4 pad 15: unconnected-(U4-A0-Pad15) -> +3V3
- U4 pad 16: unconnected-(U4-A1-Pad16) -> GND
- U4 pad 17: unconnected-(U4-A2-Pad17) -> GND
- U4 pad 18: unconnected-(U4-~{RESET}-Pad18) -> Net-(U4-~{RESET})
- U4 pad 21: /IN3_1_L -> /IN4_1_L
- U4 pad 22: /IN3_2_L -> /IN3_1_L
- U4 pad 23: /IN4_1_L -> /IN4_2_L
- U4 pad 24: /IN4_2_L -> /IN3_2_L
Routing:
- net /IN4_1_L: track 0.00 -> 75.6 mm, vias 0 -> 1
- net /IN3_1_L: track 0.00 -> 72.6 mm
- net /IN4_2_L: track 0.00 -> 72.4 mm, vias 0 -> 1
- net /IN3_2_L: track 0.00 -> 68.9 mm
- net Net-(D7-Pad2): track 0.00 -> 32.6 mm
- net /M2_A: track 0.00 -> 30.4 mm, vias 0 -> 1
- net unconnected-(D7-Pad2): track 27.6 -> 0.00 mm
- net Net-(D7-Pad3): track 0.00 -> 27.4 mm
- net unconnected-(D7-Pad3): track 24.3 -> 0.00 mm
- net GND: track 297.5 -> 320.4 mm, vias 10 -> 12
- net +3V3: track 65.2 -> 79.7 mm, vias 5 -> 11
- net /M1_A: track 0.91 -> 10.5 mm, vias 0 -> 1

Commit message: update
Parts:
- added U16: ESP32-DevKitC, PCM_Espressif:ESP32-DevKitC, F.Cu at (1.56, 7.07)
- moved R30 3.33 mm to (207.1, 95.4), turned to 90 degrees
- moved R29 3.02 mm to (212.8, 95.5), turned to 90 degrees

Commit message: update
Parts:
- added R31: R0603_4.7k_1%_100mW_100PPM_AC, Resistor_SMD:R_0603_1608Metric, F.Cu at (242.9, 66.4)
- added R32: R0603_4.7k_1%_100mW_100PPM_AC, Resistor_SMD:R_0603_1608Metric, F.Cu at (242.9, 68.9)
- added R33: R0805_1.5k_1%_125mW_100PPM_AC, Resistor_SMD:R_0805_2012Metric, F.Cu at (247.1, 73.2)
- added R34: R0805_1.5k_1%_125mW_100PPM_AC, Resistor_SMD:R_0805_2012Metric, F.Cu at (247.1, 76.2)
- added R35: R0805_1.5k_1%_125mW_100PPM_AC, Resistor_SMD:R_0805_2012Metric, F.Cu at (247.1, 79.2)
- added R36: R0805_1.5k_1%_125mW_100PPM_AC, Resistor_SMD:R_0805_2012Metric, F.Cu at (247.1, 82.1)
- added R37: R0603_4.7k_1%_100mW_100PPM_AC, Resistor_SMD:R_0603_1608Metric, F.Cu at (242.9, 71.4)
- added R38: R0603_4.7k_1%_100mW_100PPM_AC, Resistor_SMD:R_0603_1608Metric, F.Cu at (242.9, 73.9)
- added R39: R0603_4.7k_1%_100mW_100PPM_AC, Resistor_SMD:R_0603_1608Metric, F.Cu at (242.9, 76.4)
- added R40: R0603_4.7k_1%_100mW_100PPM_AC, Resistor_SMD:R_0603_1608Metric, F.Cu at (242.9, 78.9)
- added U17: LTV-817S, Package_DIP:SMDIP-4_W9.53mm, F.Cu at (251.5, 68.5)
- U16: value ESP32-DevKitC -> LTV-817S; footprint PCM_Espressif:ESP32-DevKitC -> Package_DIP:SMDIP-4_W9.53mm
Connections:
- MOD1 pad C10: unconnected-(MOD1-PadC10) -> GND2
- MOD1 pad C11: unconnected-(MOD1-PadC11) -> /OWIRE
- MOD1 pad C12: unconnected-(MOD1-PadC12) -> +3V3
- U16 pad 1: unconnected-(U16-3V3-Pad1) -> Net-(R33-Pad2)
- U16 pad 2: unconnected-(U16-CHIP_PU-Pad2) -> Net-(R34-Pad2)
- U16 pad 3: unconnected-(U16-SENSOR_VP/GPIO36/ADC1_CH0-Pad3) -> GND
- U16 pad 4: unconnected-(U16-SENSOR_VN/GPIO39/ADC1_CH3-Pad4) -> /IN5_1_L
- U2 pad 1: unconnected-(U2-GPB0-Pad1) -> /IN5_1_L
- U2 pad 2: unconnected-(U2-GPB1-Pad2) -> /IN5_2_L

Commit message: update
Parts:
- added D8: SM4007, Diode_SMD:D_MELF, B.Cu at (112.5, 103.0)
- added D9: SM4007, Diode_SMD:D_MELF, B.Cu at (128.9, 103.2)
- added K7: SANYOU_SRD_Form_C, Relay_THT:Relay_SPDT_SANYOU_SRD_Series_Form_C, F.Cu at (112.4, 98.9)
- added K8: SANYOU_SRD_Form_C, Relay_THT:Relay_SPDT_SANYOU_SRD_Series_Form_C, F.Cu at (128.7, 99.0)
- moved U16 161.6 mm to (139.8, 90.7), turned to -90 degrees
- moved U17 108.3 mm to (145.5, 90.7), turned to -90 degrees
- moved U2 67.0 mm to (188.0, 105.0)
Connections:
- MOD1 pad D1: unconnected-(MOD1-PadD1) -> +24V
- MOD1 pad D10: unconnected-(MOD1-PadD10) -> /NC1
- MOD1 pad D2: unconnected-(MOD1-PadD2) -> /IN5_2_P
- MOD1 pad D3: unconnected-(MOD1-PadD3) -> +24V
- MOD1 pad D4: unconnected-(MOD1-PadD4) -> /IN5_1_P
- MOD1 pad D5: unconnected-(MOD1-PadD5) -> /NO2
- MOD1 pad D6: unconnected-(MOD1-PadD6) -> /COM2
- MOD1 pad D7: unconnected-(MOD1-PadD7) -> /NC2
- MOD1 pad D8: unconnected-(MOD1-PadD8) -> /NO1
- MOD1 pad D9: unconnected-(MOD1-PadD9) -> /COM1
Routing:
- net /COM2: track 0.00 -> 27.2 mm
- net /COM1: track 0.00 -> 26.6 mm
- net /NO2: track 0.00 -> 13.5 mm
- net /NO1: track 0.00 -> 12.9 mm
- net /NC2: track 0.00 -> 12.6 mm
- net /NC1: track 0.00 -> 12.0 mm

Commit message: update
Parts:
- added C3: 100nF, Capacitor_THT:C_Disc_D5.0mm_W2.5mm_P5.00mm, F.Cu at (246.0, 126.0)
- added C4: 100uF, Capacitor_THT:CP_Radial_D8.0mm_P3.50mm, F.Cu at (247.6, 109.7)
- added C5: 100uF, Capacitor_THT:CP_Radial_D8.0mm_P3.50mm, F.Cu at (247.6, 119.2)
- added C6: 100nF, Capacitor_THT:C_Disc_D5.0mm_W2.5mm_P5.00mm, F.Cu at (246.0, 130.1)
- added J3: Conn_01x05_Pin, Connector_JST:JST_EH_B6B-EH-A_1x06_P2.50mm_Vertical, F.Cu at (151.2, 97.9)
- added J4: Conn_01x05_Pin, Connector_JST:JST_EH_B6B-EH-A_1x06_P2.50mm_Vertical, F.Cu at (157.1, 97.9)
- added U18: R-78E3.3-1.0, Converter_DCDC:Converter_DCDC_RECOM_R-78E-0.5_THT, F.Cu at (166.9, 87.1)
- moved R34 109.3 mm to (138.0, 82.8), turned to -90 degrees
- moved R33 106.4 mm to (141.1, 82.8), turned to -90 degrees
- moved R36 102.8 mm to (144.3, 82.8), turned to 90 degrees
- moved R35 100.4 mm to (146.8, 82.8), turned to -90 degrees
Routing:
- net +24V: track 325.2 -> 419.2 mm
- net Net-(U14-Vin-): track 7.39 -> 30.3 mm
- net /nREL2: track 0.00 -> 8.59 mm
- net /nREL1: track 0.00 -> 7.96 mm
- net +3V3: track 79.7 -> 76.9 mm, vias 11 -> 12

Commit message: update
Parts:
- added C7: 100nF, Capacitor_SMD:C_0603_1608Metric, F.Cu at (152.5, 117.0)
- added C8: 100nF, Capacitor_SMD:C_0603_1608Metric, F.Cu at (136.8, 116.1)
- added JP1: Jumper_2_Bridged, Jumper:SolderJumper-2_P1.3mm_Open_RoundedPad1.0x1.5mm, B.Cu at (200.7, 70.1)
- moved R32 104.9 mm to (142.5, 99.4), turned to 180 degrees
- moved R31 102.3 mm to (146.1, 99.4)
- moved R37 75.7 mm to (170.1, 92.3), turned to 180 degrees
- moved R39 74.8 mm to (170.1, 93.8), turned to 180 degrees
- moved R38 74.7 mm to (170.1, 90.8), turned to 180 degrees
- moved R40 70.7 mm to (173.2, 90.8)
- moved U2 5.35 mm to (188.0, 110.3)
- moved U4 0.20 mm to (148.8, 110.3)
- moved R27 0.15 mm to (154.1, 103.5)
Connections:
- C5 pad 1: VBUS -> +24V
- C6 pad 1: VBUS -> +24V
- J3 pad 6: VBUS -> +24V
- J4 pad 6: VBUS -> +24V
- MOD1 pad C10: GND2 -> GND
- U18 pad 1: VBUS -> +24V
Routing:
- net +3V3: track 76.9 -> 147.5 mm, vias 12 -> 13
- net /SCL: track 38.7 -> 77.7 mm, vias 3 -> 4
- net /SDA: track 38.4 -> 75.9 mm, vias 1 -> 2
- net /INT: track 0.00 -> 33.1 mm
- net +24V: track 419.2 -> 445.5 mm
- net GND2: track 0.00 -> 19.2 mm
- net /OWIRE: track 0.00 -> 19.1 mm
- net /SIG_CLOSE: track 0.00 -> 9.49 mm
- net /SIG_OPEN: track 0.00 -> 9.29 mm
- net GND: track 320.4 -> 327.8 mm, vias 12 -> 19
- net /M1_A: track 10.5 -> 9.57 mm
- added copper zone on B.Cu, net Net-(U14-Vin-)
- added copper zone on B.Cu, net Net-(U3-Vin-)

Commit message: update
Connections:
- U2 pad 3: unconnected-(U2-GPB2-Pad3) -> /REL1
- U5 pad 1: unconnected-(U5-I1-Pad1) -> /REL1
- U5 pad 16: unconnected-(U5-O1-Pad16) -> /nREL1
Routing:
- net /nREL1: track 7.96 -> 18.6 mm, vias 0 -> 1
