File: pcb/ESPhome_greenhouse_controller.kicad_pcb (KiCad board)
At the start: 2 copper layers, 135.7 x 83 mm, 88 parts, among them J3 Conn_01x05_Pin, J4 Conn_01x05_Pin, K1 SANYOU_SRD_Form_C, K2 SANYOU_SRD_Form_C, K3 SANYOU_SRD_Form_C, K4 SANYOU_SRD_Form_C, K5 SANYOU_SRD_Form_C, K6 SANYOU_SRD_Form_C, K7 SANYOU_SRD_Form_C, K8 SANYOU_SRD_Form_C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

Commit message: update
Parts:
- added C10: 100nF, Capacitor_SMD:C_0603_1608Metric, F.Cu at (168.8, 116.0)
- added C9: 100nF, Capacitor_SMD:C_0603_1608Metric, F.Cu at (190.9, 117.1)
- added JP2: Jumper_2_Bridged, Jumper:SolderJumper-2_P1.3mm_Open_RoundedPad1.0x1.5mm, B.Cu at (155.1, 142.2)
- moved R28 39.7 mm to (193.6, 103.5)
- moved R27 1.63 mm to (152.4, 103.6), turned to 0 degrees
- moved C7 1.00 mm to (151.5, 117.0)
- moved R10 0.12 mm to (104.2, 117.4)
- turned R36 to -90 degrees
Connections:
- MOD1 pad E1: (no net) -> +24V
- MOD1 pad E2: (no net) -> MOTOR
- R1 pad 1: +24V -> MOTOR
- R2 pad 1: +24V -> MOTOR
- U14 pad 10: +24V -> MOTOR
- U14 pad 8: +24V -> MOTOR
- U2 pad 4: unconnected-(U2-GPB3-Pad4) -> /REL2
- U2 pad 5: unconnected-(U2-GPB4-Pad5) -> /nSIG_CLOSE
- U2 pad 6: unconnected-(U2-GPB5-Pad6) -> /nSIG_OPEN
- U3 pad 10: +24V -> MOTOR
- U3 pad 8: +24V -> MOTOR
Routing:
- net MOTOR: track 0.00 -> 91.4 mm, vias 0 -> 3
- net /REL1: track 0.00 -> 77.2 mm
- net /IN5_2_L: track 0.00 -> 54.1 mm, vias 0 -> 2
- net /IN5_1_L: track 0.00 -> 53.9 mm, vias 0 -> 2
- net /REL2: track 0.00 -> 40.8 mm
- net GND: track 327.8 -> 361.1 mm, vias 19 -> 70
- net /SDA: track 75.9 -> 106.9 mm, vias 2 -> 5
- net /INT: track 33.1 -> 63.9 mm
- net /SCL: track 77.7 -> 106.7 mm, vias 4 -> 5
- net +24V: track 445.5 -> 424.5 mm
- net /nSIG_CLOSE: track 0.00 -> 16.8 mm
- net /nSIG_OPEN: track 0.00 -> 15.3 mm
- net /IN5_1_P: track 0.00 -> 14.7 mm
- net +3V3: track 147.5 -> 162.1 mm, vias 13 -> 16
- net unconnected-(U2-GPB6-Pad7): track 0.00 -> 14.0 mm
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- added copper zone on B.Cu, net GND
- added copper zone on F.Cu, net GND
- removed copper zone on B.Cu, net +24V

Commit message: update
Parts:
- added Q1: BC817, Package_TO_SOT_SMD:SOT-23, F.Cu at (1.95, 1.90)
- U5: value ULN2003A -> ULN2803A; footprint Package_SO:SOIC-16W_5.3x10.2mm_P1.27mm -> Package_SO:SOIC-18W_7.5x11.6mm_P1.27mm
- moved U5 1.13 mm to (113.4, 111.8)
Connections:
- U5 pad 1: /REL1 -> unconnected-(U5-I1-Pad1)
- U5 pad 10: /nSOUND -> +24V
- U5 pad 11: /nFWD1 -> /nSOUND
- U5 pad 12: /nREV1 -> /nFWD1
- U5 pad 13: /nREV2 -> /nREV1
- U5 pad 14: /nFWD2 -> /nREV2
- U5 pad 15: /nLIGHT -> /nFWD2
- U5 pad 16: /nREL1 -> /nLIGHT
- U5 pad 2: /LIGHT -> /REL1
- U5 pad 3: /FWD2 -> /LIGHT
- U5 pad 4: /REV2 -> /FWD2
- U5 pad 5: /REV1 -> /REV2
- U5 pad 6: /FWD1 -> /REV1
- U5 pad 7: /SOUND -> /FWD1
- U5 pad 8: GND -> /SOUND
- U5 pad 9: +24V -> GND
Routing:
- net unconnected-(U5-O1-Pad18): track 0.00 -> 17.2 mm, vias 0 -> 1
- net GND: track 361.1 -> 352.1 mm, vias 70 -> 62
- net /IN1_2_L: track 59.5 -> 66.2 mm
- net /IN1_1_L: track 62.3 -> 68.0 mm
- net /IN2_1_L: track 58.9 -> 64.5 mm
- net /IN2_2_L: track 54.5 -> 59.6 mm
- net /nREL1: track 28.2 -> 24.8 mm
- net /SOUND: track 36.7 -> 40.0 mm
- net /M2_A: track 30.0 -> 27.8 mm
- net /LIGHT: track 33.2 -> 35.3 mm
- net /REL1: track 77.2 -> 79.2 mm
- net /FWD2: track 36.3 -> 38.1 mm
- net /REV2: track 39.5 -> 41.1 mm
- net /FWD1: track 45.4 -> 46.9 mm
- net /REV1: track 42.5 -> 44.0 mm
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
Commit message: update
Parts:
- removed C5: 100uF, Capacitor_THT:CP_Radial_D8.0mm_P3.50mm
- added J1: Conn_01x05_Pin, Connector_PinHeader_2.54mm:PinHeader_1x05_P2.54mm_Vertical, F.Cu at (180.0, 88.3)
- C3, C6: footprint Capacitor_THT:C_Disc_D5.0mm_W2.5mm_P5.00mm -> Capacitor_SMD:C_0805_2012Metric
- moved C6 96.4 mm to (161.4, 83.8), turned to 90 degrees
- moved C3 83.5 mm to (167.8, 96.7), turned to 90 degrees
- moved C4 77.1 mm to (171.3, 98.7)
Connections:
- MOD1 pad C5: unconnected-(MOD1-PadC5) -> /1
- MOD1 pad C6: unconnected-(MOD1-PadC6) -> /2
- MOD1 pad C7: unconnected-(MOD1-PadC7) -> /3
- MOD1 pad C8: unconnected-(MOD1-PadC8) -> /4
- MOD1 pad C9: unconnected-(MOD1-PadC9) -> /5
- U2 pad 21: unconnected-(U2-GPA0-Pad21) -> /1
- U2 pad 22: unconnected-(U2-GPA1-Pad22) -> /2
- U2 pad 23: unconnected-(U2-GPA2-Pad23) -> /3
- U2 pad 24: unconnected-(U2-GPA3-Pad24) -> /4
- U2 pad 25: unconnected-(U2-GPA4-Pad25) -> /5
- U2 pad 26: unconnected-(U2-GPA5-Pad26) -> /6
- U2 pad 27: unconnected-(U2-GPA6-Pad27) -> /7
- U2 pad 7: unconnected-(U2-GPB6-Pad7) -> /8
- U5 pad 1: unconnected-(U5-I1-Pad1) -> /REL2
- U5 pad 18: unconnected-(U5-O1-Pad18) -> /nREL2
Routing:
- net +3V3: track 162.0 -> 311.9 mm, vias 16 -> 22
- net /8: track 0.00 -> 44.3 mm, vias 0 -> 3
- net /REL2: track 40.8 -> 80.2 mm, vias 0 -> 2
- net /1: track 0.00 -> 35.0 mm
- net /5: track 0.00 -> 33.8 mm
- net /2: track 0.00 -> 33.5 mm
- net /4: track 0.00 -> 32.2 mm
- net /3: track 0.00 -> 32.0 mm
- net /nSIG_CLOSE: track 16.8 -> 43.4 mm, vias 0 -> 2
- net /nSIG_OPEN: track 15.3 -> 36.6 mm, vias 0 -> 2
- net /nREL2: track 8.59 -> 26.0 mm, vias 0 -> 1
- net /6: track 0.00 -> 17.4 mm
- net unconnected-(U5-O1-Pad18): track 17.2 -> 0.00 mm, vias 1 -> 0
- net /7: track 0.00 -> 14.1 mm
- net unconnected-(U2-GPB6-Pad7): track 14.0 -> 0.00 mm
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- added copper zone on B.Cu, net GND2
- added copper zone on F.Cu, net GND2

Commit message: update
Parts:
- removed J1: Conn_01x05_Pin, Connector_PinHeader_2.54mm:PinHeader_1x05_P2.54mm_Vertical
- removed Q1: BC817, Package_TO_SOT_SMD:SOT-23
- added J2: Conn_01x05_Pin, Connector_JST:JST_EH_B6B-EH-A_1x06_P2.50mm_Vertical, F.Cu at (180.0, 86.0)
Routing:
- net +3V3: track 311.9 -> 320.4 mm
- net /OWIRE: track 19.1 -> 25.1 mm, vias 0 -> 1

Commit message: update
Parts:
- removed R27, R28: R0603_4.7k_1%_100mW_100PPM_AC, Resistor_SMD:R_0603_1608Metric
- removed U4: MCP23017_SO, Package_SO:SOIC-28W_7.5x17.9mm_P1.27mm
- added U19: TCA9555DBR, Package_SO:SSOP-24_5.3x8.2mm_P0.65mm, F.Cu at (184.1, 111.3)
- U2: value MCP23017_SO -> TCA9555DBR; footprint Package_SO:SOIC-28W_7.5x17.9mm_P1.27mm -> Package_SO:SSOP-24_5.3x8.2mm_P0.65mm
- moved C9 52.6 mm to (139.6, 105.3), turned to 180 degrees
- moved U2 42.4 mm to (145.6, 109.3)
- moved C7 28.1 mm to (178.0, 107.7), turned to 180 degrees
- moved J2 0.20 mm to (180.2, 86.0)
Connections:
- U2 pad 1: /IN5_1_L -> /INT
- U2 pad 10: GND -> /REV1
- U2 pad 11: unconnected-(U2-NC-Pad11) -> /FWD1
- U2 pad 12: /SCL -> GND
- U2 pad 13: /SDA -> /IN4_1_L
- U2 pad 14: unconnected-(U2-NC-Pad14) -> /IN3_1_L
- U2 pad 15: GND -> /IN4_2_L
- U2 pad 16: GND -> /IN3_2_L
- U2 pad 17: GND -> /M2_A
- U2 pad 18: Net-(U2-~{RESET}) -> /IN2_1_L
- U2 pad 19: /INT -> /IN1_1_L
- U2 pad 2: /IN5_2_L -> GND
- U2 pad 20: /INT -> /SOUND
- U2 pad 21: /1 -> +3V3
- U2 pad 22: /2 -> /SCL
- U2 pad 23: /3 -> /SDA
- U2 pad 24: /4 -> +3V3
- U2 pad 3: /REL1 -> GND
- U2 pad 4: /REL2 -> /M1_A
- U2 pad 5: /nSIG_CLOSE -> /IN2_2_L
- U2 pad 6: /nSIG_OPEN -> /IN1_2_L
- U2 pad 7: /8 -> /LIGHT
- U2 pad 8: unconnected-(U2-GPB7-Pad8) -> /FWD2
- U2 pad 9: +3V3 -> /REV2
Routing:
- net +3V3: track 320.4 -> 303.8 mm, vias 22 -> 20
- net /8: track 44.3 -> 31.5 mm
- net /INT: track 77.5 -> 85.4 mm, vias 0 -> 3
- net /REL2: track 80.2 -> 73.6 mm
- net /SCL: track 106.7 -> 112.2 mm
- net /IN5_1_L: track 53.8 -> 59.4 mm
- net /REL1: track 78.5 -> 73.4 mm, vias 0 -> 2
- net GND: track 352.1 -> 347.3 mm, vias 81 -> 83
- net /M1_A: track 9.57 -> 14.3 mm
- net /SOUND: track 40.1 -> 44.4 mm
- net /IN1_1_L: track 68.0 -> 71.7 mm
- net /LIGHT: track 35.3 -> 38.9 mm
- net /FWD2: track 38.1 -> 41.4 mm
- net /IN2_1_L: track 64.5 -> 67.7 mm
- net /REV2: track 41.1 -> 43.8 mm
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